File: BLCD_BerdAir.kicad_pcb (KiCad board)
At the start: 4 copper layers, 40 x 55 mm, 70 parts, among them IC1 MCT8316A1VRGFR, IC2 MCT8316A1VRGFR, J1 Screw_Terminal_01x03, J2 Screw_Terminal_01x03, J3 Screw_Terminal_01x03, J4 Conn_02x12_Odd_Even, J5 Conn_01x02_Pin, J6 Conn_01x02_Pin, J7 Conn_02x06_Top_Bottom

Commit message: tested
Connections:
- net /ESC/VDDA renamed /ESC_A/VDDA
- net /ESC1/VDDA renamed /ESC_B/VDDA
