File: BLCD_BerdAir.kicad_sch (KiCad schematic)
At the start: 32 parts, among them J1 Screw_Terminal_01x03, J4 Conn_02x12_Odd_Even, J7 Conn_02x06_Top_Bottom

Commit message: tested
Parts:
- renumbered J1 to J3
Other:
- sheet ESC renamed ESC_A
- sheet ESC1 renamed ESC_B
