File: MCT8316AV.kicad_sch (KiCad schematic)
At the start: 19 parts, among them IC1 MCT8316A1VRGFR, J1 Screw_Terminal_01x03, J5 Conn_01x02_Pin

Commit message: tested
Parts:
- renumbered C6 to C15, C3 to C7, R6 to R2, R6 to R35, R6 to R37, R6 to R39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
Other:
- note added: "NC"
- note added: "SOX"
- moved on the sheet: R35
